Commit message: add bumper

File: turtlebot3_description/urdf/robot.gazebo.xacro (robot description, xacro)
@@ -4,4 +4,5 @@
   <xacro:arg name="imu_visual"   default="false"/>
   <xacro:arg name="camera_visual" default="true"/>
+  <!-- <xacro:arg name="cover_visual" default="true"/> -->
   <xacro:arg name="r200_cam_rgb_px" default="0.005"/>
   <xacro:arg name="r200_cam_rgb_py" default="0.018"/>
@@ -169,3 +170,12 @@
     </sensor>
   </gazebo>
+  <gazebo reference="cover_link">
+   <sensor name='my_contact' type='contact'>
+       <plugin name="my_plugin" filename="libcontact.so"/>
+          <contact>
+            <collision>bumper_collision_collision</collision>
+          </contact>
+        <update_rate> 5 </update_rate>
+        </sensor>
+  </gazebo>
 </robot>

File: turtlebot3_description/urdf/robot.urdf.xacro (robot description, xacro)
@@ -61,15 +61,15 @@
       <origin xyz="-0.032 0 -0.12" rpy="1.5708 0 1.5708"/>
       <geometry>
-        <!-- <cylinder length="0.2" radius="0.225"/> -->
+        <!-- <mesh filename="package://robotino_description/meshes/bumper.stl" scale="0.001 0.001 0.001"/> -->
         <mesh filename="package://robotino_description/meshes/robotino_body_diy.stl" scale="0.001 0.001 0.001"/>
       </geometry>
       <material name="light_black"/>
     </visual>
-    <!-- <collision>
-      <origin xyz="-0.032 0 0.17" rpy="0 0 0"/>
+    <collision name="bumper_collision">
+      <origin xyz="-0.032 0 -0.1" rpy="1.5708 0 1.5708"/>
       <geometry>
-        <cylinder length="0.325" radius="0.45"/>
+        <mesh filename="package://robotino_description/meshes/bumper.stl" scale="0.001 0.001 0.001"/>
       </geometry>
-    </collision> -->
+    </collision>
     <inertial>
       <origin xyz="0 0 0" rpy="0 0 0"/>

Commit message: update bumper sensor before fix

File: turtlebot3_description/urdf/robot.gazebo.xacro (robot description, xacro)
@@ -171,8 +171,10 @@
   </gazebo>
   <gazebo reference="cover_link">
-   <sensor name='my_contact' type='contact'>
-       <plugin name="my_plugin" filename="libcontact.so"/>
+   <sensor name='bumper_contact' type='contact'>
+   <always_on>true</always_on>
+       <plugin name="my_plugin" filename="libgazebo_ros_bumper.so"/>
+       <!-- <plugin name="my_plugin" filename="libcontact.so"/> -->
           <contact>
-            <collision>bumper_collision_collision</collision>
+            <collision>bumper_collision</collision>
           </contact>
         <update_rate> 5 </update_rate>
