Commit message: finalisasi prototype robotino

File: turtlebot3_description/urdf/robot.urdf.xacro (robot description, xacro)
@@ -11,7 +11,8 @@
   <link name="camera_link">
     <visual name="camera">
-      <origin xyz="0 0 0" rpy="0 0 0"/>
+      <origin xyz="0 0 0" rpy="1.5708 0 1.5708"/>
       <geometry>
-        <box size="0.02 0.07 0.03" />
+        <!-- <box size="0.02 0.07 0.03" /> -->
+        <mesh filename="package://robotino_description/meshes/Intel_Realsense_D435.stl" scale="0.001 0.001 0.001"/>
       </geometry>
     </visual>
@@ -31,5 +32,5 @@
     <parent link="base_link"/>
     <child link="camera_link"/>
-    <origin xyz="0 0 0.25" rpy="0 0 0"/>
+    <origin xyz="0 0 0.3" rpy="0 0 0"/>
     <axis xyz="0 0 0"/>
   </joint>
@@ -58,7 +59,8 @@
    <link name="cover_link">
     <visual>
-      <origin xyz="-0.032 0 0" rpy="0 0 0"/>
+      <origin xyz="-0.032 0 -0.12" rpy="1.5708 0 1.5708"/>
       <geometry>
-        <cylinder length="0.2" radius="0.225"/>
+        <!-- <cylinder length="0.2" radius="0.225"/> -->
+        <mesh filename="package://robotino_description/meshes/robotino_body_diy.stl" scale="0.001 0.001 0.001"/>
       </geometry>
       <material name="light_black"/>
@@ -72,8 +74,8 @@
     <inertial>
       <origin xyz="0 0 0" rpy="0 0 0"/>
-      <mass value="0.01"/>
-      <inertia ixx="0.01" ixy="0.0" ixz="0.0"
-               iyy="0.01" iyz="0.0"
-               izz="0.01" />
+      <mass value="0.0001"/>
+      <inertia ixx="0.001" ixy="0.0" ixz="0.0"
+               iyy="0.001" iyz="0.0"
+               izz="0.001" />
     </inertial>
   </link>
@@ -169,5 +171,5 @@
     <parent link="base_link"/>
     <child link="base_scan"/>
-    <origin xyz="-0.032 0 0.05" rpy="0 0 0"/>
+    <origin xyz="-0.032 0 0.03" rpy="0 0 0"/>
   </joint>
   <link name="base_scan">

Commit message: fixing robot joint

File: turtlebot3_description/urdf/robot.urdf.xacro (robot description, xacro)
@@ -80,5 +80,5 @@
     </inertial>
   </link>
-  <joint name="cover_joint" type="continuous">
+  <joint name="cover_joint" type="fixed">
     <parent link="base_link"/>
     <child link="cover_link"/>

Commit message: try to solve the coliision problem but not yet solved lol, im stuck. trying to transform the environment file to my own

File: turtlebot3_description/urdf/robot.urdf.xacro (robot description, xacro)
@@ -2,5 +2,5 @@
 <robot name="turtlebot3_burger" xmlns:xacro="http://ros.org/wiki/xacro">
   <xacro:include filename="$(find turtlebot3_description)/urdf/common_properties.xacro"/>
-  <xacro:include filename="$(find turtlebot3_description)/urdf/robot.gazebo.xacro"/>
+  <xacro:include filename="$(find turtlebot3_description)/urdf/robotutil.gazebo.xacro"/>
   <link name="base_footprint"/>
   <joint name="base_joint" type="fixed">

File: turtlebot3_description/urdf/robotutil.gazebo.xacro (robot description, xacro)
@@ -171,13 +171,16 @@
   </gazebo>
   <gazebo reference="cover_link">
-   <sensor name='bumper_contact' type='contact'>
-   <always_on>true</always_on>
-       <plugin name="my_plugin" filename="libgazebo_ros_bumper.so"/>
+    <sensor name='bumper_contact' type='contact'>
+      <always_on>true</always_on>
+      <plugin name="my_plugin" filename="libgazebo_ros_bumper.so">
+        <bumperTopicName>bumper_contact</bumperTopicName>
+        <frameName>bumper</frameName>
+      </plugin>
        <!-- <plugin name="my_plugin" filename="libcontact.so"/> -->
-          <contact>
-            <collision>bumper_collision</collision>
-          </contact>
-        <update_rate> 5 </update_rate>
-        </sensor>
+        <contact>
+          <collision>base_footprint_fixed_joint_lump__bumper_collision_collision_3</collision>
+        </contact>
+        <update_rate> 1000 </update_rate>
+    </sensor>
   </gazebo>
 </robot>
