Commit message: move worskapce to a real folder

File: robotino_description/urdf/robot.urdf.xacro (robot description, xacro)
@@ -2,5 +2,5 @@
 <robot name="turtlebot3_burger" xmlns:xacro="http://ros.org/wiki/xacro">
   <xacro:include filename="$(find turtlebot3_description)/urdf/common_properties.xacro"/>
-  <xacro:include filename="$(find turtlebot3_description)/urdf/robotutil.gazebo.xacro"/>
+  <xacro:include filename="$(find turtlebot3_description)/urdf/robotoutil.gazebo.xacro"/>
   <link name="base_footprint"/>
   <joint name="base_joint" type="fixed">
@@ -219,6 +219,6 @@
   <joint name="bumper_joint" type="fixed">
     <parent link="base_link"/>
-    <child link="bumper"/>
-    <origin xyz="-0.032 0 0.03" rpy="0 0 0"/>
+    <child link="bumper_scan"/>
+    <origin xyz="-0.032 0 0.035" rpy="0 0 0"/>
   </joint>
 </robot>

Commit message: delete unecessary file

File: robotino_description/urdf/robot.urdf.xacro (robot description, xacro)
@@ -1,4 +1,4 @@
 <!-- Edited by: Ihsan Nurkhotib -->
-<!-- if you editing, please place your name below -->
+<!-- if you editing this file, please place your name below -->
 <?xml version="1.0" ?>
 <robot name="robotino" xmlns:xacro="http://ros.org/wiki/xacro">
@@ -15,5 +15,4 @@
       <origin xyz="0 0 0" rpy="1.5708 0 1.5708"/>
       <geometry>
-        <!-- <box size="0.02 0.07 0.03" /> -->
         <mesh filename="package://robotino_description/meshes/Intel_Realsense_D435.stl" scale="0.001 0.001 0.001"/>
       </geometry>
@@ -63,5 +62,4 @@
       <origin xyz="-0.032 0 -0.12" rpy="1.5708 0 1.5708"/>
       <geometry>
-        <!-- <mesh filename="package://robotino_description/meshes/bumper.stl" scale="0.001 0.001 0.001"/> -->
         <mesh filename="package://robotino_description/meshes/robotino_body_diy.stl" scale="0.001 0.001 0.001"/>
       </geometry>

File: robotino_description/urdf/robotutil.gazebo.xacro (robot description, xacro)
@@ -1,4 +1,4 @@
 <!-- Edited by: Ihsan Nurkhotib -->
-<!-- if you editing, please place your name below -->
+<!-- if you editing this file, please place your name below -->
 <?xml version="1.0"?>
 <robot name="turtlebot3_burger_sim" xmlns:xacro="http://ros.org/wiki/xacro">
